Commit message: fix(model): hand_mount includes the real flange->palm offset (dz = -2.5 cm)
The user found a 2.5 cm adapter plate in the physical TCP->XHand
assembly. Live verification (FoundationPose cube x board extrinsic vs
URDF-FK rest position) showed the real palm sits 2.5 cm CLOSER along
the flange axis than the URDF modelled — sign empirically pinned by
A/B: +0.025 doubled the y-residual to 43 mm, -0.025 collapsed ALL axes
to (10, 7, 4) mm. Note: fingertip obs are palm-relative and unaffected;
this fixes the env-frame anchoring that auto-center had been silently
absorbing. Pick-task USD still carries the old mount (flagged, not
touched — trained policies depend on it).

Co-Authored-By: Claude Fable 5 <noreply@anthropic.com>

File: source/xhand_inhand/xhand_inhand/assets/xarm7_xhand/xarm7_xhand.urdf (robot description, URDF)
Before this commit: robot xarm7_xhand, 22 links, 21 joints
Joints:
- joint hand_mount: origin xyz=0 0 0 rpy=0 0 4.71239 -> xyz=0 0 -0.025 rpy=0 0 4.71239

Commit message: fix(model): hand_mount dz = +0.025 — the 2.5 cm TCP adapter plate, final
Per the physical assembly (user-confirmed): flange -> 2.5 cm plate ->
XHand. Supersedes the -0.025 experiment; the plate is rendered as a
disk between flange and palm in the live viewer.

Co-Authored-By: Claude Fable 5 <noreply@anthropic.com>

File: source/xhand_inhand/xhand_inhand/assets/xarm7_xhand/xarm7_xhand.urdf (robot description, URDF)
Before this commit: robot xarm7_xhand, 22 links, 21 joints
Joints:
- joint hand_mount: origin xyz=0 0 -0.025 rpy=0 0 4.71239 -> xyz=0 0 0.025 rpy=0 0 4.71239

Commit message: fix(model): TCP adapter plate finalized at 2.0 cm (live-render verified)
User-tuned against the one-lib live view (FoundationPose cube vs FK
hand): 2.0 cm matches the physical assembly.

Co-Authored-By: Claude Fable 5 <noreply@anthropic.com>

File: source/xhand_inhand/xhand_inhand/assets/xarm7_xhand/xarm7_xhand.urdf (robot description, URDF)
Before this commit: robot xarm7_xhand, 22 links, 21 joints
Joints:
- joint hand_mount: origin xyz=0 0 0.025 rpy=0 0 4.71239 -> xyz=0 0 0.020 rpy=0 0 4.71239
